File: hardware/dwtk-ice-mega/dwtk-ice-mega.kicad_pcb (KiCad board)
At the start: 2 copper layers, 68.6 x 39.4 mm, 34 parts, among them J1 USB_B_Mini, J2 Conn_01x02_Female, J3 Conn_01x02_Female, J4 AVR-ISP-6, J5 AVR-ISP-10, Q1 BC548, U1 ATmega88PA-PU, Y1 Crystal 20MHz

Commit message: hardware: update dwtk-ice-mega pcb values
Parts:
- C1: value 10uF -> 10u
- C2: value 100nF -> 100n
- C3, C4: value 22pF -> 22p
- D1, D2: value D_Zener -> 3,6
- D3: value LED -> Red
- D4: value LED -> Green
- H1: value Conn_01x03 -> Jumper
- J1: value USB_B_Mini -> USB B Mini Female
- J2, J3: value Conn_01x02_Female -> JST XH2P Female
- R1, R2: value 68R -> 68
- R10, R11, R7, R8, R9: value 470R -> 470
- Y1: value Crystal 20MHz -> 20.0000 MHz
