File: hardware/dwtk-ice-mega/dwtk-ice-mega.sch (KiCad schematic (older format))
At the start: 28 parts, among them J1 USB B Mini Female, J2 JST XH2P Female, J3 JST XH2P Female, J4 AVR-ISP-6, J5 AVR-ISP-10, Q1 BC548, U1 ATmega88PA-PU, Y1 20.0000 MHz

Commit message: hardware: added mouser references
Parts:
- C1: Mouser Ref. (none) -> 667-ECA-1VM100I
- C2: Mouser Ref. (none) -> 594-K104K15X7RF53K2
- C3, C4: Mouser Ref. (none) -> 594-K220J15C0GF53L2
- D1, D2: Mouser Ref. (none) -> 512-BZX79C3V6
- D3: Mouser Ref. (none) -> 604-WP710A10SEC/J3
- D4: Mouser Ref. (none) -> 604-WP710A10ZGC/G
- H1: Mouser Ref. (none) -> 68797-236HLF
- J1: Mouser Ref. (none) -> 538-54819-0519
- J2, J3: Mouser Ref. (none) -> N/A
- J4: Mouser Ref. (none) -> 710-61200621621
- J5: Mouser Ref. (none) -> 710-61201021621
- Q1: Mouser Ref. (none) -> 821-BC548B-A1
- R1, R2: Mouser Ref. (none) -> 291-68-RC
- R10, R11, R7, R8, R9: Mouser Ref. (none) -> 291-470-RC
- R3: Mouser Ref. (none) -> 291-2.2K-RC
- R4, R5: Mouser Ref. (none) -> 291-1.5K-RC
- R6: Mouser Ref. (none) -> 291-22K-RC
- U1: Mouser Ref. (none) -> 556-ATMEGA88PA-PU
- Y1: Mouser Ref. (none) -> 815-ABL-20-B4Y
Changed lines of the file:
@@
 F 3 "~" H 5200 4700 50  0001 C CNN
 F 4 "RND 205-00862" H 5050 4750 50  0001 C CNN "Reichelt Ref."
+F 5 "538-54819-0519" H 5050 4750 50  0001 C CNN "Mouser Ref."
 	1    5050 4750
 	-1   0    0    -1
@@
 F 3 "~" H 3200 4750 50  0001 C CNN
 F 4 "1/4W 68" H 3200 4750 50  0001 C CNN "Reichelt Ref."
+F 5 "291-68-RC" H 3200 4750 50  0001 C CNN "Mouser Ref."
 	1    3200 4750
 	0    1    -1   0
@@
 F 3 "~" H 3650 4850 50  0001 C CNN
 F 4 "1/4W 68" H 3650 4850 50  0001 C CNN "Reichelt Ref."
+F 5 "291-68-RC" H 3650 4850 50  0001 C CNN "Mouser Ref."
 	1    3650 4850
 	0    1    1    0
@@
 F 3 "~" H 4300 5400 50  0001 C CNN
 F 4 "ZF 3,6" H 4300 5400 50  0001 C CNN "Reichelt Ref."
+F 5 "512-BZX79C3V6" H 4300 5400 50  0001 C CNN "Mouser Ref."
 	1    4300 5400
 	0    1    1    0
@@
 F 3 "~" H 3650 4950 50  0001 C CNN
 F 4 "1/4W 2,2K" H 3650 4950 50  0001 C CNN "Reichelt Ref."
+F 5 "291-2.2K-RC" H 3650 4950 50  0001 C CNN "Mouser Ref."
 	1    3650 4950
 	0    1    1    0
@@
 F 3 "~" H 3800 5400 50  0001 C CNN
 F 4 "ZF 3,6" H 3800 5400 50  0001 C CNN "Reichelt Ref."
+F 5 "512-BZX79C3V6" H 3800 5400 50  0001 C CNN "Mouser Ref."
 	1    3800 5400
 	0    1    1    0
@@
 F 3 "~" H 2850 6050 50  0001 C CNN
 F 4 "RND 135-00155" H 2850 6050 50  0001 C CNN "Reichelt Ref."
+F 5 "604-WP710A10SEC/J3" H 2850 6050 50  0001 C CNN "Mouser Ref."
 	1    2850 6050
 	0    -1   -1   0
@@
 F 3 "~" H 2850 5600 50  0001 C CNN
 F 4 "1/4W 1,5K" H 2850 5600 50  0001 C CNN "Reichelt Ref."
+F 5 "291-1.5K-RC" H 2850 5600 50  0001 C CNN "Mouser Ref."
 	1    2850 5600
 	1    0    0    -1
@@
 F 3 "~" H 1250 2900 50  0001 C CNN
 F 4 "1/4W 1,5K" H 1250 2900 50  0001 C CNN "Reichelt Ref."
+F 5 "291-1.5K-RC" H 1250 2900 50  0001 C CNN "Mouser Ref."
 	1    1250 2900
 	1    0    0    -1
@@
 F 3 "~" H 1250 3350 50  0001 C CNN
 F 4 "RND 135-00157" H 1250 3350 50  0001 C CNN "Reichelt Ref."
+F 5 "604-WP710A10ZGC/G" H 1250 3350 50  0001 C CNN "Mouser Ref."
 	1    1250 3350
 	0    -1   -1   0
@@
 F 3 "~" H 3800 3750 50  0001 C CNN
 F 4 "KERKO 22P" H 3800 3750 50  0001 C CNN "Reichelt Ref."
+F 5 "594-K220J15C0GF53L2" H 3800 3750 50  0001 C CNN "Mouser Ref."
 	1    3800 3750
 	0    1    1    0
@@
 F 3 "~" H 3400 4200 50  0001 C CNN
 F 4 "JST XH2P ST" H 3400 4200 50  0001 C CNN "Reichelt Ref."
+F 5 "N/A" H 3400 4200 50  0001 C CNN "Mouser Ref."
 	1    3400 4200
 	1    0    0    1
@@
 F 3 "http://www.fairchildsemi.com/ds/BC/BC547.pdf" H 6500 4200 50  0001 L CNN
 F 4 "BC 548B" H 6500 4200 50  0001 C CNN "Reichelt Ref."
+F 5 "821-BC548B-A1" H 6500 4200 50  0001 C CNN "Mouser Ref."
 	1    6500 4200
 	1    0    0    -1
@@
 F 3 "~" H 6350 4600 50  0001 C CNN
 F 4 "1/4W 470" H 6350 4600 50  0001 C CNN "Reichelt Ref."
+F 5 "291-470-RC" H 6350 4600 50  0001 C CNN "Mouser Ref."
 	1    6350 4600
 	0    1    1    0
@@
 F 3 "~" H 6300 3600 50  0001 C CNN
 F 4 "1/4W 22K" H 6300 3600 50  0001 C CNN "Reichelt Ref."
+F 5 "291-22K-RC" H 6300 3600 50  0001 C CNN "Mouser Ref."
 	1    6300 3600
 	1    0    0    -1
@@
 F 3 "~" H 7400 3350 50  0001 C CNN
 F 4 "JST XH2P ST" H 7400 3350 50  0001 C CNN "Reichelt Ref."
+F 5 "N/A" H 7400 3350 50  0001 C CNN "Mouser Ref."
 	1    7400 3350
 	1    0    0    -1
@@
 F 3 " ~" H 8475 2650 50  0001 C CNN
 F 4 "WSL 6G" H 9750 3200 50  0001 C CNN "Reichelt Ref."
+F 5 "710-61200621621" H 9750 3200 50  0001 C CNN "Mouser Ref."
 	1    9750 3200
 	-1   0    0    -1
@@
 F 3 " ~" H 8475 4000 50  0001 C CNN
 F 4 "WSL 10G" H 9750 4550 50  0001 C CNN "Reichelt Ref."
+F 5 "710-61201021621" H 9750 4550 50  0001 C CNN "Mouser Ref."
 	1    9750 4550
 	-1   0    0    -1
@@
 F 3 "~" H 8700 3100 50  0001 C CNN
 F 4 "1/4W 470" H 8700 3100 50  0001 C CNN "Reichelt Ref."
+F 5 "291-470-RC" H 8700 3100 50  0001 C CNN "Mouser Ref."
 	1    8700 3100
 	0    1    1    0
@@
 F 3 "~" H 8250 3200 50  0001 C CNN
 F 4 "1/4W 470" H 8250 3200 50  0001 C CNN "Reichelt Ref."
+F 5 "291-470-RC" H 8250 3200 50  0001 C CNN "Mouser Ref."
 	1    8250 3200
 	0    1    1    0
@@
 F 3 "http://ww1.microchip.com/downloads/en/DeviceDoc/ATmega48PA_88PA_168PA-Data-Sheet-40002011A.pdf" H 2200 4050 50  0001 C CNN
 F 4 "ATMEGA 88PA-PU" H 2200 4050 50  0001 C CNN "Reichelt Ref."
+F 5 "556-ATMEGA88PA-PU" H 2200 4050 50  0001 C CNN "Mouser Ref."
 	1    2200 4050
 	1    0    0    -1
@@
 F 3 "~" H 3350 3550 50  0001 C CNN
 F 4 "20,0000-HC49U-S" H 3350 3550 50  0001 C CNN "Reichelt Ref."
+F 5 "815-ABL-20-B4Y" H 3350 3550 50  0001 C CNN "Mouser Ref."
 	1    3350 3550
 	0    1    1    0
@@
 F 3 "~" H 3800 3250 50  0001 C CNN
 F 4 "KERKO 22P" H 3800 3250 50  0001 C CNN "Reichelt Ref."
+F 5 "594-K220J15C0GF53L2" H 3800 3250 50  0001 C CNN "Mouser Ref."
 	1    3800 3250
 	0    1    1    0
@@
 F 3 "~" H 2900 2650 50  0001 C CNN
 F 4 "1/4W 470" H 2900 2650 50  0001 C CNN "Reichelt Ref."
+F 5 "291-470-RC" H 2900 2650 50  0001 C CNN "Mouser Ref."
 	1    2900 2650
 	1    0    0    -1
@@
 F 3 "~" H 1500 1950 50  0001 C CNN
 F 4 "RAD 10/35" H 1500 1950 50  0001 C CNN "Reichelt Ref."
+F 5 "667-ECA-1VM100I" H 1500 1950 50  0001 C CNN "Mouser Ref."
 	1    1500 1950
 	1    0    0    -1
@@
 F 3 "~" H 1950 1950 50  0001 C CNN
 F 4 "KERKO 100N" H 1950 1950 50  0001 C CNN "Reichelt Ref."
+F 5 "594-K104K15X7RF53K2" H 1950 1950 50  0001 C CNN "Mouser Ref."
 	1    1950 1950
 	1    0    0    -1
@@
 F 3 "~" H 7800 2350 50  0001 C CNN
 F 4 "SL 1X40G 2,54" H 7800 2350 50  0001 C CNN "Reichelt Ref."
+F 5 "68797-236HLF" H 7800 2350 50  0001 C CNN "Mouser Ref."
 	1    7800 2350
 	1    0    0    -1
@@
 F 3 "~" H 4200 4100 50  0001 C CNN
 F 4 "1/4W 470" H 4200 4100 50  0001 C CNN "Reichelt Ref."
+F 5 "291-470-RC" H 4200 4100 50  0001 C CNN "Mouser Ref."
 	1    4200 4100
 	1    0    0    -1
