File: hardware/dwtk-ice/dwtk-ice.sch (KiCad schematic (older format))
At the start: 27 parts, among them J1 USB B Mini Female, J2 JST XH2P Female, J3 JST XH2P Female, J4 AVR-ISP-6, J5 AVR-ISP-10, Q1 BC548, U1 ATtiny4313-PU, Y1 20.0000 MHz

Commit message: hardware: added mouser references
Parts:
- C1: Mouser Ref. (none) -> 667-ECA-1VM100I
- C2: Mouser Ref. (none) -> 594-K104K15X7RF53K2
- C3, C4: Mouser Ref. (none) -> 594-K220J15C0GF53L2
- D1, D2: Mouser Ref. (none) -> 512-BZX79C3V6
- D3: Mouser Ref. (none) -> 604-WP710A10SEC/J3
- D4: Mouser Ref. (none) -> 604-WP710A10ZGC/G
- H1: Mouser Ref. (none) -> 68797-236HLF
- J1: Mouser Ref. (none) -> 538-54819-0519
- J2, J3: Mouser Ref. (none) -> N/A
- J4: Mouser Ref. (none) -> 710-61200621621
- J5: Mouser Ref. (none) -> 710-61201021621
- Q1: Mouser Ref. (none) -> 821-BC548B-A1
- R1, R2: Mouser Ref. (none) -> 291-68-RC
- R10, R7, R8, R9: Mouser Ref. (none) -> 291-470-RC
- R3: Mouser Ref. (none) -> 291-2.2K-RC
- R4, R5: Mouser Ref. (none) -> 291-1.5K-RC
- R6: Mouser Ref. (none) -> 291-22K-RC
- U1: Mouser Ref. (none) -> 556-ATTINY4313-PU
- Y1: Mouser Ref. (none) -> 815-ABL-20-B4Y
Changed lines of the file:
@@
 F 3 "~" H 2200 2600 50  0001 C CNN
 F 4 "RND 205-00862" H 2050 2650 50  0001 C CNN "Reichelt Ref."
+F 5 "538-54819-0519" H 2050 2650 50  0001 C CNN "Mouser Ref."
 	1    2050 2650
 	1    0    0    -1
@@
 F 3 "http://ww1.microchip.com/downloads/en/DeviceDoc/doc8246.pdf" H 3950 4250 50  0001 C CNN
 F 4 "ATTINY 4313 PU" H 3950 4250 50  0001 C CNN "Reichelt Ref."
+F 5 "556-ATTINY4313-PU" H 3950 4250 50  0001 C CNN "Mouser Ref."
 	1    3950 4250
 	1    0    0    -1
@@
 F 3 "~" H 4950 4550 50  0001 C CNN
 F 4 "1/4W 68" H 4950 4550 50  0001 C CNN "Reichelt Ref."
+F 5 "291-68-RC" H 4950 4550 50  0001 C CNN "Mouser Ref."
 	1    4950 4550
 	0    1    1    0
@@
 F 3 "~" H 5250 4650 50  0001 C CNN
 F 4 "1/4W 68" H 5250 4650 50  0001 C CNN "Reichelt Ref."
+F 5 "291-68-RC" H 5250 4650 50  0001 C CNN "Mouser Ref."
 	1    5250 4650
 	0    1    1    0
@@
 F 3 "~" H 6050 5000 50  0001 C CNN
 F 4 "ZF 3,6" H 6050 5000 50  0001 C CNN "Reichelt Ref."
+F 5 "512-BZX79C3V6" H 6050 5000 50  0001 C CNN "Mouser Ref."
 	1    6050 5000
 	0    1    1    0
@@
 F 3 "~" H 5250 4750 50  0001 C CNN
 F 4 "1/4W 2,2K" H 5250 4750 50  0001 C CNN "Reichelt Ref."
+F 5 "291-2.2K-RC" H 5250 4750 50  0001 C CNN "Mouser Ref."
 	1    5250 4750
 	0    1    1    0
@@
 F 3 "~" H 5550 5000 50  0001 C CNN
 F 4 "ZF 3,6" H 5550 5000 50  0001 C CNN "Reichelt Ref."
+F 5 "512-BZX79C3V6" H 5550 5000 50  0001 C CNN "Mouser Ref."
 	1    5550 5000
 	0    1    1    0
@@
 F 3 "~" H 5050 5500 50  0001 C CNN
 F 4 "RND 135-00155" H 5050 5500 50  0001 C CNN "Reichelt Ref."
+F 5 "604-WP710A10SEC/J3" H 5050 5500 50  0001 C CNN "Mouser Ref."
 	1    5050 5500
 	0    -1   -1   0
@@
 F 3 "~" H 5050 5150 50  0001 C CNN
 F 4 "1/4W 1,5K" H 5050 5150 50  0001 C CNN "Reichelt Ref."
+F 5 "291-1.5K-RC" H 5050 5150 50  0001 C CNN "Mouser Ref."
 	1    5050 5150
 	1    0    0    -1
@@
 F 3 "~" H 4700 5150 50  0001 C CNN
 F 4 "1/4W 1,5K" H 4700 5150 50  0001 C CNN "Reichelt Ref."
+F 5 "291-1.5K-RC" H 4700 5150 50  0001 C CNN "Mouser Ref."
 	1    4700 5150
 	1    0    0    -1
@@
 F 3 "~" H 4700 5500 50  0001 C CNN
 F 4 "RND 135-00157" H 4700 5500 50  0001 C CNN "Reichelt Ref."
+F 5 "604-WP710A10ZGC/G" H 4700 5500 50  0001 C CNN "Mouser Ref."
 	1    4700 5500
 	0    -1   -1   0
@@
 F 3 "~" H 2500 3900 50  0001 C CNN
 F 4 "20,0000-HC49U-S" H 2500 3900 50  0001 C CNN "Reichelt Ref."
+F 5 "815-ABL-20-B4Y" H 2500 3900 50  0001 C CNN "Mouser Ref."
 	1    2500 3900
 	0    1    1    0
@@
 F 3 "~" H 2150 3650 50  0001 C CNN
 F 4 "KERKO 22P" H 2150 3650 50  0001 C CNN "Reichelt Ref."
+F 5 "594-K220J15C0GF53L2" H 2150 3650 50  0001 C CNN "Mouser Ref."
 	1    2150 3650
 	0    1    1    0
@@
 F 3 "~" H 2150 4150 50  0001 C CNN
 F 4 "KERKO 22P" H 2150 4150 50  0001 C CNN "Reichelt Ref."
+F 5 "594-K220J15C0GF53L2" H 2150 4150 50  0001 C CNN "Mouser Ref."
 	1    2150 4150
 	0    1    1    0
@@
 F 3 "~" H 5300 2050 50  0001 C CNN
 F 4 "KERKO 100N" H 5300 2050 50  0001 C CNN "Reichelt Ref."
+F 5 "594-K104K15X7RF53K2" H 5300 2050 50  0001 C CNN "Mouser Ref."
 	1    5300 2050
 	1    0    0    -1
@@
 F 3 "~" H 4850 2050 50  0001 C CNN
 F 4 "RAD 10/35" H 4850 2050 50  0001 C CNN "Reichelt Ref."
+F 5 "667-ECA-1VM100I" H 4850 2050 50  0001 C CNN "Mouser Ref."
 	1    4850 2050
 	1    0    0    -1
@@
 F 3 "~" H 1950 1950 50  0001 C CNN
 F 4 "JST XH2P ST" H 1950 1950 50  0001 C CNN "Reichelt Ref."
+F 5 "N/A" H 1950 1950 50  0001 C CNN "Mouser Ref."
 	1    1950 1950
 	-1   0    0    1
@@
 F 3 "http://www.fairchildsemi.com/ds/BC/BC547.pdf" H 5950 4050 50  0001 L CNN
 F 4 "BC 548B" H 5950 4050 50  0001 C CNN "Reichelt Ref."
+F 5 "821-BC548B-A1" H 5950 4050 50  0001 C CNN "Mouser Ref."
 	1    5950 4050
 	1    0    0    -1
@@
 F 3 "~" H 5850 4300 50  0001 C CNN
 F 4 "1/4W 470" H 5850 4300 50  0001 C CNN "Reichelt Ref."
+F 5 "291-470-RC" H 5850 4300 50  0001 C CNN "Mouser Ref."
 	1    5850 4300
 	0    1    1    0
@@
 F 3 "~" H 5750 3450 50  0001 C CNN
 F 4 "1/4W 22K" H 5750 3450 50  0001 C CNN "Reichelt Ref."
+F 5 "291-22K-RC" H 5750 3450 50  0001 C CNN "Mouser Ref."
 	1    5750 3450
 	1    0    0    -1
@@
 F 3 "~" H 6850 3200 50  0001 C CNN
 F 4 "JST XH2P ST" H 6850 3200 50  0001 C CNN "Reichelt Ref."
+F 5 "N/A" H 6850 3200 50  0001 C CNN "Mouser Ref."
 	1    6850 3200
 	1    0    0    -1
@@
 F 3 "~" H 6600 4550 50  0001 C CNN
 F 4 "1/4W 470" H 6600 4550 50  0001 C CNN "Reichelt Ref."
+F 5 "291-470-RC" H 6600 4550 50  0001 C CNN "Mouser Ref."
 	1    6600 4550
 	1    0    0    -1
@@
 F 3 " ~" H 7925 2500 50  0001 C CNN
 F 4 "WSL 6G" H 9200 3050 50  0001 C CNN "Reichelt Ref."
+F 5 "710-61200621621" H 9200 3050 50  0001 C CNN "Mouser Ref."
 	1    9200 3050
 	-1   0    0    -1
@@
 F 3 " ~" H 7925 3850 50  0001 C CNN
 F 4 "WSL 10G" H 9200 4400 50  0001 C CNN "Reichelt Ref."
+F 5 "710-61201021621" H 9200 4400 50  0001 C CNN "Mouser Ref."
 	1    9200 4400
 	-1   0    0    -1
@@
 F 3 "~" H 8150 2950 50  0001 C CNN
 F 4 "1/4W 470" H 8150 2950 50  0001 C CNN "Reichelt Ref."
+F 5 "291-470-RC" H 8150 2950 50  0001 C CNN "Mouser Ref."
 	1    8150 2950
 	0    1    1    0
@@
 F 3 "~" H 7700 3050 50  0001 C CNN
 F 4 "1/4W 470" H 7700 3050 50  0001 C CNN "Reichelt Ref."
+F 5 "291-470-RC" H 7700 3050 50  0001 C CNN "Mouser Ref."
 	1    7700 3050
 	0    1    1    0
@@
 F 3 "~" H 7250 2300 50  0001 C CNN
 F 4 "SL 1X40G 2,54" H 7250 2300 50  0001 C CNN "Reichelt Ref."
+F 5 "68797-236HLF" H 7250 2300 50  0001 C CNN "Mouser Ref."
 	1    7250 2300
 	1    0    0    -1
