File: hardware/dwtk-ice-lite/dwtk-ice-lite.sch (KiCad schematic (older format))
At the start: 21 parts, among them J1 USB B Mini Female, J2 JST XH2P Female, J3 JST XH2P Female, Q1 BC548, U1 ATtiny4313-PU, Y1 20.0000 MHz

Commit message: hardware: added mouser references
Parts:
- C1: Mouser Ref. (none) -> 667-ECA-1VM100I
- C2: Mouser Ref. (none) -> 594-K104K15X7RF53K2
- C3, C4: Mouser Ref. (none) -> 594-K220J15C0GF53L2
- D1, D2: Mouser Ref. (none) -> 512-BZX79C3V6
- D3: Mouser Ref. (none) -> 604-WP710A10SEC/J3
- D4: Mouser Ref. (none) -> 604-WP710A10ZGC/G
- J1: Mouser Ref. (none) -> 538-54819-0519
- J2, J3: Mouser Ref. (none) -> N/A
- Q1: Mouser Ref. (none) -> 821-BC548B-A1
- R1, R2: Mouser Ref. (none) -> 291-68-RC
- R3: Mouser Ref. (none) -> 291-2.2K-RC
- R4, R5: Mouser Ref. (none) -> 291-1.5K-RC
- R6: Mouser Ref. (none) -> 291-22K-RC
- R7: Mouser Ref. (none) -> 291-470-RC
- U1: Mouser Ref. (none) -> 556-ATTINY4313-PU
- Y1: Mouser Ref. (none) -> 815-ABL-20-B4Y
Changed lines of the file:
@@
 F 3 "~" H 3550 2550 50  0001 C CNN
 F 4 "RND 205-00862" H 3400 2600 50  0001 C CNN "Reichelt Ref."
+F 5 "538-54819-0519" H 3400 2600 50  0001 C CNN "Mouser Ref."
 	1    3400 2600
 	1    0    0    -1
@@
 F 3 "http://ww1.microchip.com/downloads/en/DeviceDoc/doc8246.pdf" H 5300 4200 50  0001 C CNN
 F 4 "ATTINY 4313 PU" H 5300 4200 50  0001 C CNN "Reichelt Ref."
+F 5 "556-ATTINY4313-PU" H 5300 4200 50  0001 C CNN "Mouser Ref."
 	1    5300 4200
 	1    0    0    -1
@@
 F 3 "~" H 6300 4500 50  0001 C CNN
 F 4 "1/4W 68" H 6300 4500 50  0001 C CNN "Reichelt Ref."
+F 5 "291-68-RC" H 6300 4500 50  0001 C CNN "Mouser Ref."
 	1    6300 4500
 	0    1    1    0
@@
 F 3 "~" H 6600 4600 50  0001 C CNN
 F 4 "1/4W 68" H 6600 4600 50  0001 C CNN "Reichelt Ref."
+F 5 "291-68-RC" H 6600 4600 50  0001 C CNN "Mouser Ref."
 	1    6600 4600
 	0    1    1    0
@@
 F 3 "~" H 7400 4950 50  0001 C CNN
 F 4 "ZF 3,6" H 7400 4950 50  0001 C CNN "Reichelt Ref."
+F 5 "512-BZX79C3V6" H 7400 4950 50  0001 C CNN "Mouser Ref."
 	1    7400 4950
 	0    1    1    0
@@
 F 3 "~" H 6600 4700 50  0001 C CNN
 F 4 "1/4W 2,2K" H 6600 4700 50  0001 C CNN "Reichelt Ref."
+F 5 "291-2.2K-RC" H 6600 4700 50  0001 C CNN "Mouser Ref."
 	1    6600 4700
 	0    1    1    0
@@
 F 3 "~" H 6900 4950 50  0001 C CNN
 F 4 "ZF 3,6" H 6900 4950 50  0001 C CNN "Reichelt Ref."
+F 5 "512-BZX79C3V6" H 6900 4950 50  0001 C CNN "Mouser Ref."
 	1    6900 4950
 	0    1    1    0
@@
 F 3 "~" H 6400 5450 50  0001 C CNN
 F 4 "RND 135-00155" H 6400 5450 50  0001 C CNN "Reichelt Ref."
+F 5 "604-WP710A10SEC/J3" H 6400 5450 50  0001 C CNN "Mouser Ref."
 	1    6400 5450
 	0    -1   -1   0
@@
 F 3 "~" H 6400 5100 50  0001 C CNN
 F 4 "1/4W 1,5K" H 6400 5100 50  0001 C CNN "Reichelt Ref."
+F 5 "291-1.5K-RC" H 6400 5100 50  0001 C CNN "Mouser Ref."
 	1    6400 5100
 	1    0    0    -1
@@
 F 3 "~" H 6050 5100 50  0001 C CNN
 F 4 "1/4W 1,5K" H 6050 5100 50  0001 C CNN "Reichelt Ref."
+F 5 "291-1.5K-RC" H 6050 5100 50  0001 C CNN "Mouser Ref."
 	1    6050 5100
 	1    0    0    -1
@@
 F 3 "~" H 6050 5450 50  0001 C CNN
 F 4 "RND 135-00157" H 6050 5450 50  0001 C CNN "Reichelt Ref."
+F 5 "604-WP710A10ZGC/G" H 6050 5450 50  0001 C CNN "Mouser Ref."
 	1    6050 5450
 	0    -1   -1   0
@@
 F 3 "~" H 3900 3850 50  0001 C CNN
 F 4 "20,0000-HC49U-S" H 3900 3850 50  0001 C CNN "Reichelt Ref."
+F 5 "815-ABL-20-B4Y" H 3900 3850 50  0001 C CNN "Mouser Ref."
 	1    3900 3850
 	0    1    1    0
@@
 F 3 "~" H 3550 3600 50  0001 C CNN
 F 4 "KERKO 22P" H 3550 3600 50  0001 C CNN "Reichelt Ref."
+F 5 "594-K220J15C0GF53L2" H 3550 3600 50  0001 C CNN "Mouser Ref."
 	1    3550 3600
 	0    1    1    0
@@
 F 3 "~" H 3550 4100 50  0001 C CNN
 F 4 "KERKO 22P" H 3550 4100 50  0001 C CNN "Reichelt Ref."
+F 5 "594-K220J15C0GF53L2" H 3550 4100 50  0001 C CNN "Mouser Ref."
 	1    3550 4100
 	0    1    1    0
@@
 F 3 "~" H 5850 2150 50  0001 C CNN
 F 4 "RAD 10/35" H 5850 2150 50  0001 C CNN "Reichelt Ref."
+F 5 "667-ECA-1VM100I" H 5850 2150 50  0001 C CNN "Mouser Ref."
 	1    5850 2150
 	1    0    0    -1
@@
 F 3 "~" H 3300 1900 50  0001 C CNN
 F 4 "JST XH2P ST" H 3300 1900 50  0001 C CNN "Reichelt Ref."
+F 5 "N/A" H 3300 1900 50  0001 C CNN "Mouser Ref."
 	1    3300 1900
 	-1   0    0    1
@@
 F 3 "http://www.fairchildsemi.com/ds/BC/BC547.pdf" H 7300 4000 50  0001 L CNN
 F 4 "BC 548B" H 7300 4000 50  0001 C CNN "Reichelt Ref."
+F 5 "821-BC548B-A1" H 7300 4000 50  0001 C CNN "Mouser Ref."
 	1    7300 4000
 	1    0    0    -1
@@
 F 3 "~" H 7150 4400 50  0001 C CNN
 F 4 "1/4W 470" H 7150 4400 50  0001 C CNN "Reichelt Ref."
+F 5 "291-470-RC" H 7150 4400 50  0001 C CNN "Mouser Ref."
 	1    7150 4400
 	0    1    1    0
@@
 F 3 "~" H 7100 3400 50  0001 C CNN
 F 4 "1/4W 22K" H 7100 3400 50  0001 C CNN "Reichelt Ref."
+F 5 "291-22K-RC" H 7100 3400 50  0001 C CNN "Mouser Ref."
 	1    7100 3400
 	1    0    0    -1
@@
 F 3 "~" H 8200 3150 50  0001 C CNN
 F 4 "JST XH2P ST" H 8200 3150 50  0001 C CNN "Reichelt Ref."
+F 5 "N/A" H 8200 3150 50  0001 C CNN "Mouser Ref."
 	1    8200 3150
 	1    0    0    -1
@@
 F 3 "~" H 6500 2150 50  0001 C CNN
 F 4 "KERKO 100N" H 6500 2150 50  0001 C CNN "Reichelt Ref."
+F 5 "594-K104K15X7RF53K2" H 6500 2150 50  0001 C CNN "Mouser Ref."
 	1    6500 2150
 	1    0    0    -1
